Commit message: Add files via upload

File: quadruped.urdf (robot description, URDF)
Before this commit: robot quadruped, 5 links, 4 joints
Links:
- added link BL_hip, mass 0.2; collision cylinder length=0.1 radius=0.02; visual cylinder length=0.1 radius=0.02
- added link BR_hip, mass 0.2; collision cylinder length=0.1 radius=0.02; visual cylinder length=0.1 radius=0.02
- added link FL_hip, mass 0.2; collision cylinder length=0.1 radius=0.02; visual cylinder length=0.1 radius=0.02
- added link FR_hip, mass 0.2; collision cylinder length=0.1 radius=0.02; visual cylinder length=0.1 radius=0.02
- link BL_leg: mass 0.5 -> 1.5; geometry collision cylinder length=0.25 radius=0.025; visual cylinder length=0.25 radius=0.025
- link BR_leg: mass 0.5 -> 1.5; geometry collision cylinder length=0.25 radius=0.025; visual cylinder length=0.25 radius=0.025
- link FL_leg: mass 0.5 -> 1.5; geometry collision cylinder length=0.25 radius=0.025; visual cylinder length=0.25 radius=0.025
- link FR_leg: mass 0.5 -> 1.5; geometry collision cylinder length=0.25 radius=0.025; visual cylinder length=0.25 radius=0.025
- link base_link: mass 5.0 -> 10.0; geometry collision box size=0.4 0.2 0.1; visual box size=0.4 0.2 0.1
Joints:
- added joint BL_hip_joint: type revolute, parent base_link, child BL_hip, origin xyz=-0.2 0.1 -0.02 rpy=0 0 0, axis 1 0 0, limit lower=-0.3 upper=0.3 effort=1000 velocity=10.0
- added joint BR_hip_joint: type revolute, parent base_link, child BR_hip, origin xyz=-0.2 -0.1 -0.02 rpy=0 0 0, axis 1 0 0, limit lower=-0.3 upper=0.3 effort=1000 velocity=10.0
- added joint FL_hip_joint: type revolute, parent base_link, child FL_hip, origin xyz=0.2 0.1 -0.02 rpy=0 0 0, axis 1 0 0, limit lower=-0.3 upper=0.3 effort=1000 velocity=10.0
- added joint FR_hip_joint: type revolute, parent base_link, child FR_hip, origin xyz=0.2 -0.1 -0.02 rpy=0 0 0, axis 1 0 0, limit lower=-0.3 upper=0.3 effort=1000 velocity=10.0
- joint BL_joint: limit lower=-1.57 upper=1.57 effort=10 velocity=1.0 -> lower=-1.57 upper=1.57 effort=1000 velocity=10.0; origin xyz=-0.15 0.1 0 rpy=0 0 0 -> xyz=0 0.1 -0.02 rpy=0 0 0; parent base_link -> BL_hip
- joint BR_joint: limit lower=-1.57 upper=1.57 effort=10 velocity=1.0 -> lower=-1.57 upper=1.57 effort=1000 velocity=10.0; origin xyz=-0.15 -0.1 0 rpy=0 0 0 -> xyz=0 -0.1 -0.02 rpy=0 0 0; parent base_link -> BR_hip
- joint FL_joint: limit lower=-1.57 upper=1.57 effort=10 velocity=1.0 -> lower=-1.57 upper=1.57 effort=1000 velocity=10.0; origin xyz=0.15 0.1 0 rpy=0 0 0 -> xyz=0 0.1 -0.02 rpy=0 0 0; parent base_link -> FL_hip
- joint FR_joint: limit lower=-1.57 upper=1.57 effort=10 velocity=1.0 -> lower=-1.57 upper=1.57 effort=1000 velocity=10.0; origin xyz=0.15 -0.1 0 rpy=0 0 0 -> xyz=0 -0.1 -0.02 rpy=0 0 0; parent base_link -> FR_hip
